Commit message: added class names for OD training, vision dependencies in Dockerfile, transformation to base_link for 3d localization; finalized PC gen and deleted camera_depth_optical_frame in xacro because of conflicting names with the realsense camera driver's TF tree

File: src/bcr_arm/bcr_arm_description/urdf/sensors/depth_camera.urdf.xacro (robot description, xacro)
@@ -25,20 +25,4 @@
       </inertial>
     </link>
-    <!-- Camera Sensor Link -->
-    <joint name="${prefix}camera_joint" type="fixed">
-      <parent link="${prefix}camera_base_link"/>
-      <child link="${prefix}camera_link"/>
-      <!-- Pointing forward from the mount -->
-      <origin xyz="0.0125 0 0" rpy="0 0 0"/>
-    </joint>
-    <link name="${prefix}camera_link"/>
-    <!-- Camera Optical Frame -->
-    <joint name="${prefix}camera_optical_joint" type="fixed">
-      <parent link="${prefix}camera_link"/>
-      <child link="${prefix}camera_depth_optical_frame"/>
-      <!-- Standard ROS optical frame rotation -->
-      <origin xyz="0 0 0" rpy="${-pi/2} 0 ${-pi/2}"/>
-    </joint>
-    <link name="${prefix}camera_depth_optical_frame"/>
     <!-- Ignition Gazebo Camera Plugin -->
     <gazebo reference="${prefix}camera_link">
